File: kicad/twin-round-display/ev-gauge-twin-round-display.kicad_sch (KiCad schematic)
At the start: 0 parts

Commit message: Add first-pass schematic for twin round display board
ESP32-S3-MINI-1 with TCAN332 CAN transceiver, TPS54202 buck and
AP2127K 3.3V LDO, USB-C, PC817 opto input, TVS/polyfuse protection
and display/expansion headers. PCB layout not started.

Co-Authored-By: Claude Opus 5.5 <noreply@anthropic.com>
Parts:
- added C1: C, Capacitor_SMD:C_1206_3216Metric, symbol Device:C
- added C10, C8: 10uF, Capacitor_SMD:C_0603_1608Metric, symbol Device:C
- added C11, C12: 1uF, Capacitor_SMD:C_0603_1608Metric, symbol Device:C
- added C2, C3: 22uF, Capacitor_SMD:C_0805_2012Metric, symbol Device:C
- added C4: C, Capacitor_SMD:C_0603_1608Metric, symbol Device:C
- added C5, C6, C7, C9, C_BOOT: 100nF, Capacitor_SMD:C_0603_1608Metric, symbol Device:C
- added D1: D_TVS, Diode_SMD:D_SMB, symbol Device:D_TVS
- added D2: D_TVS, Package_TO_SOT_SMD:SOT-23, symbol Device:D_TVS
- added D3: D_Schottky, symbol Device:D_Schottky
- added D4: 1N4148W, Diode_SMD:D_SOD-123, symbol Device:D
- added F1: 500mA, Fuse:Fuse_1812_4532Metric, symbol Device:Polyfuse
- added F2: 100mA, Fuse:Fuse_1206_3216Metric, symbol Device:Polyfuse
- added J1: USB_C_Receptacle_USB2.0_14P, Connector_USB:USB_C_Receptacle_XKB_U262-16X1B41, symbol Connector:USB_C_Receptacle_USB2.0_14P
- added J2: Conn_01x05_Socket, symbol Connector:Conn_01x05_Socket
- added J3: Conn_01x11_Socket, Connector_PinHeader_2.54mm:PinHeader_1x11_P2.54mm_Vertical, symbol Connector:Conn_01x11_Socket
- added JP1: SolderJumper_2_Open, symbol Jumper:SolderJumper_2_Open
- added L1: 10uH, Inductor_SMD:L_4x4mm, symbol Device:L
- added Q1: Q_PMOS_GSD, Package_TO_SOT_SMD:SOT-23, symbol Transistor_FET:Q_PMOS_GSD
- added Q2: Q_NMOS_GSD, Package_TO_SOT_SMD:SOT-23, symbol Transistor_FET:Q_NMOS_GSD
- added R1, R2, R5: 100k, Resistor_SMD:R_0603_1608Metric, symbol Device:R
- added R10, R9: 5.1k, Resistor_SMD:R_0603_1608Metric, symbol Device:R
- added R11: 10k, Resistor_SMD:R_0805_2012Metric, symbol Device:R
- added R12: 1k, Resistor_SMD:R_0603_1608Metric, symbol Device:R
- added R13, R4, R6: 10k, Resistor_SMD:R_0603_1608Metric, symbol Device:R
- added R3: 23.2k, Resistor_SMD:R_0603_1608Metric, symbol Device:R
- added R7: R, Resistor_SMD:R_0603_1608Metric, symbol Device:R
- added R8: 120, Resistor_SMD:R_0603_1608Metric, symbol Device:R
- added SW1, SW2: SW_Push, Button_Switch_SMD:SW_SPST_PTS645, symbol Switch:SW_Push
- added U1: ESP32-S3-MINI-1, RF_Module:ESP32-S2-MINI-1, symbol RF_Module:ESP32-S3-MINI-1
- added U2: TPS54202DDC, Package_TO_SOT_SMD:SOT-23-6, symbol Regulator_Switching:TPS54202DDC
- added U3: TCAN332, Package_SO:SOIC-8_3.9x4.9mm_P1.27mm, symbol Interface_CAN_LIN:TCAN332
- added U4: PC817, Package_DIP:DIP-4_W7.62mm, symbol Isolator:PC817
- added U5: AP2127K-3.3, Package_TO_SOT_SMD:SOT-23-5, symbol Regulator_Linear:AP2127K-3.3
Connections:
- new net: D4.1 (K), R12.2, U4.1
- new net: Q1.1 (G), R1.1
- new net: D1.1 (A1), Q1.3 (D)
- new net: C_BOOT.1, L1.1, U2.2 (SW)
- new net: Q2.1 (G), R13.1, R5.2
- new net: C11.1, D3.1 (K), U5.1 (VIN), U5.3 (EN)
- new net: C_BOOT.2, U2.6 (BOOT)
- new net: C1.1, C4.1, D1.2 (A2), D2.2 (A2), U2.3 (VIN)
- new net: F1.2, J2.1 (Pin_1)
- new net: J1.A5 (CC1), R9.1
- new net: JP1.1 (A), U3.6 (CANL)
- new net: R8.2, U3.7 (CANH)
- new net: J1.B5 (CC2), R10.1
- new net: JP1.2 (B), R8.1
- new net: F2.2, J2.4 (Pin_4)
- new net: D3.2 (A), J1.A4 (VBUS), J1.A9 (VBUS), J1.B4 (VBUS), J1.B9 (VBUS)
- new net: R2.2, R3.1, U2.4 (FB)
- new net +3.3V: C12.1, L1.2, R2.1, U1.3 (3V3), U3.3 (VCC), U5.5 (VOUT)
- new net +3V3: R11.1
- new net 12V_RAW: F1.1, Q1.2 (S)
- new net BOOT_CIRC: U1.19 (IO15)
- new net CAN_H: J2.2 (Pin_2)
- new net CAN_L: J2.3 (Pin_3)
- new net CAN_RX: U1.10 (IO6), U3.4 (RXD)
- new net CAN_TX: U1.9 (IO5), U3.1 (TXD)
- new net DN: J1.A7 (D-), J1.B7 (D-), U1.24 (USB_D+)
- new net DP: J1.A6 (D+), J1.B6 (D+), U1.23 (USB_D-)
- new net GND: C1.2, C11.2, C12.2, C4.2, D2.1 (A1), D4.2 (A), J1.A1 (GND), J1.A12 (GND), J1.B1 (GND), J1.B12 (GND), J1.SH (SHIELD), J2.5 (Pin_5), J3.1 (Pin_1), Q2.2 (S), R1.2, R10.2, R13.2, R3.2, R9.2, U1.1 (GND), U1.2 (GND), U1.42 (GND), U1.43 (GND), U1.46 (GND), U1.47 (GND), U1.48 (GND), U1.49 (GND), U1.50 (GND), U1.51 (GND), U1.52 (GND), U1.53 (GND), U1.54 (GND), U1.55 (GND), U1.56 (GND), U1.57 (GND), U1.58 (GND), U1.59 (GND), U1.60 (GND), U1.61 (GND), U1.62 (GND), U1.63 (GND), U1.64 (GND), U1.65 (GND), U2.1 (GND), U2.5 (EN), U3.2 (GND), U4.2, U4.3, U5.2 (GND)
- new net IBUS: F2.1, R12.1
- new net IBUS_RX: R11.2, U1.22 (IO18), U4.4
- new net LCD_BL: J3.10 (Pin_10), Q2.3 (D)
- new net LCD_BL_CTRL: R5.1, U1.8 (IO4)
- new net LCD_CS: J3.9 (Pin_9), U1.14 (IO10)
- new net LCD_IO0: J3.4 (Pin_4), U1.15 (IO11)
- new net LCD_IO1: J3.5 (Pin_5), U1.17 (IO13)
- new net LCD_IO2: J3.6 (Pin_6), U1.18 (IO14)
- new net LCD_IO3: J3.7 (Pin_7), U1.13 (IO9)
- new net LCD_RST: J3.8 (Pin_8), U1.20 (IO16)
- new net LCD_SCLK: J3.3 (Pin_3), U1.16 (IO12)
- new net LCD_TE: J3.11 (Pin_11), U1.25 (IO21)
- new net RES_CIRC: U1.45 (EN)
- new net VCC: J3.2 (Pin_2)
- no-connect marks 0 -> 24
